File: Mini_Solder_Iron/Mini_Solder_Iron.kicad_pcb (KiCad board)
At the start: 2 copper layers, 5 parts, among them Q1 AO4407A, U1 STM32F103C8Tx, U2 LIS2DS12, U3 SGM8557, U4 TMP36GRTZ

Commit message: update
Parts:
- added CN1: YXT-BB10-24S-02, kicad_lceda:CONN-SMD_YXT-BB10-24S-02, F.Cu at (156.5, 92.1)
- added J1: USB_C_Receptacle_USB2.0, Connector_USB:USB_C_Receptacle_HRO_TYPE-C-31-M-12, B.Cu at (167.9, 92.4)
- added U5: CH224K, kicad_lceda:ESSOP-10_L4.9-W3.9-P1.0-LS6.0-TL-EP, B.Cu at (158.3, 92.3)
- added U6: MP9942, kicad_lceda:TSOT23-8_L2.9-W1.6-P0.65-LS2.8-BL, B.Cu at (149.6, 92.4)
- moved U2 17.3 mm to (141.0, 93.0)
- moved Q1 15.8 mm to (111.2, 92.5)
- moved U1 11.7 mm to (121.7, 92.4)
- moved U4 9.84 mm to (136.4, 92.7)
- moved U3 2.75 mm to (131.5, 92.7)
Other:
- board outline added: 65 x 11 mm

Commit message: update
Parts:
- added C1: 30PF, Capacitor_SMD:C_0402_1005Metric, F.Cu at (179.4, 83.2)
- added C2: 4u7, Capacitor_SMD:C_0402_1005Metric, F.Cu at (171.8, 70.8)
- added C3: 100nf, Capacitor_SMD:C_0402_1005Metric, F.Cu at (177.5, 70.7)
- added C4: 30PF, Capacitor_SMD:C_0402_1005Metric, F.Cu at (174.9, 68.8)
- added C5: 100nf, Capacitor_SMD:C_0402_1005Metric, F.Cu at (171.8, 86.8)
- added C6: 100nf, Capacitor_SMD:C_0402_1005Metric, F.Cu at (176.5, 83.2)
- added C7: 100nf, Capacitor_SMD:C_0402_1005Metric, F.Cu at (174.6, 70.8)
- added C8: 100nf, Capacitor_SMD:C_0402_1005Metric, F.Cu at (177.8, 68.8)
- added D1: LED, LED_SMD:LED_0402_1005Metric, F.Cu at (169.1, 68.8)
- added J2: Conn_01x04, kicad_lceda:JBC245_2.4mm, F.Cu at (136.9, 92.4)
- added J3: Conn_01x04, kicad_lceda:JBC245_1.5mm, F.Cu at (150.9, 92.4)
- added J4: Conn_01x04, kicad_lceda:JBC245_3.5mm, F.Cu at (118.2, 92.4)
- added J5: Conn_01x04, kicad_lceda:JBC245_2.4mm, B.Cu at (136.9, 92.4)
- added J6: Conn_01x04, kicad_lceda:JBC245_1.5mm, B.Cu at (150.9, 92.4)
- added J7: Conn_01x04, kicad_lceda:JBC245_3.5mm, B.Cu at (118.2, 92.4)
- added JP1: SolderJumper_2_Open, Jumper:SolderJumper-2_P1.3mm_Open_RoundedPad1.0x1.5mm, F.Cu at (183.3, 87.8)
- added R1: 10K, Resistor_SMD:R_0402_1005Metric, F.Cu at (167.9, 88.5)
- added R2: 1K5, Resistor_SMD:R_0402_1005Metric, F.Cu at (168.9, 70.8)
- added R3: 10K, Resistor_SMD:R_0402_1005Metric, F.Cu at (172.0, 68.8)
- added U7: CH340E, Package_SO:MSOP-10_3x3mm_P0.5mm, B.Cu at (186.2, 92.6)
- added Y1: Crystal_GND3_Small, CSTCE8M00G55:OSC_CSTCE8M00G55-R0, F.Cu at (167.8, 92.1)
- U1: value STM32F103C8Tx -> STM32F103C8T6
- moved U1 53.0 mm to (174.7, 92.5)
- moved U2 51.5 mm to (192.5, 92.5)
- moved U4 51.4 mm to (187.8, 92.5)
- moved U3 50.8 mm to (182.3, 92.5)
- moved Q1 50.5 mm to (161.7, 92.0)
- moved CN1 43.2 mm to (199.7, 92.3)
- moved J1 42.0 mm to (209.9, 92.4)
- moved U5 42.0 mm to (200.3, 92.3)
- moved U6 42.0 mm to (191.6, 92.4)
Connections:
- U1 pad 1: unconnected-(U1-Pad1) -> +3V3
- U1 pad 10: unconnected-(U1-Pad10) -> EN1
- U1 pad 12: unconnected-(U1-Pad12) -> USART2_TX
- U1 pad 13: unconnected-(U1-Pad13) -> USART2_RX
- U1 pad 14: unconnected-(U1-Pad14) -> CS
- U1 pad 15: unconnected-(U1-Pad15) -> SCK
- U1 pad 16: unconnected-(U1-Pad16) -> MISO
- U1 pad 17: unconnected-(U1-Pad17) -> MOSI
- U1 pad 18: unconnected-(U1-Pad18) -> Button
- U1 pad 2: unconnected-(U1-Pad2) -> Net-(D1-Pad2)
- U1 pad 22: unconnected-(U1-Pad22) -> ERROR
- U1 pad 23: unconnected-(U1-Pad23) -> GND
- U1 pad 24: unconnected-(U1-Pad24) -> +3V3
- U1 pad 25: unconnected-(U1-Pad25) -> SPI2_CS
- U1 pad 26: unconnected-(U1-Pad26) -> SPI2_SCK
- U1 pad 27: unconnected-(U1-Pad27) -> SPI2_MISO
- U1 pad 28: unconnected-(U1-Pad28) -> SPI2_MOSI
- U1 pad 29: unconnected-(U1-Pad29) -> PWMA
- U1 pad 30: unconnected-(U1-Pad30) -> PWMB
- U1 pad 31: unconnected-(U1-Pad31) -> PWMC
- U1 pad 32: unconnected-(U1-Pad32) -> USB_DM
- U1 pad 33: unconnected-(U1-Pad33) -> USB_DP
- U1 pad 34: unconnected-(U1-Pad34) -> SWDIO
- U1 pad 35: unconnected-(U1-Pad35) -> GND
- U1 pad 36: unconnected-(U1-Pad36) -> +3V3
- U1 pad 37: unconnected-(U1-Pad37) -> SWCLK
- U1 pad 42: unconnected-(U1-Pad42) -> I2C1_SCL
- U1 pad 43: unconnected-(U1-Pad43) -> I2C1_SDA
- U1 pad 44: unconnected-(U1-Pad44) -> Net-(JP1-Pad2)
- U1 pad 47: unconnected-(U1-Pad47) -> GND
- U1 pad 48: unconnected-(U1-Pad48) -> +3V3
- U1 pad 5: unconnected-(U1-Pad5) -> HSE_IN
- U1 pad 6: unconnected-(U1-Pad6) -> HSE_OUT
- U1 pad 7: unconnected-(U1-Pad7) -> Net-(C6-Pad1)
- U1 pad 8: unconnected-(U1-Pad8) -> GND
- U1 pad 9: unconnected-(U1-Pad9) -> +3V3
Other:
- board size 65 x 11 mm -> 100 x 13 mm
- copper layers 2 -> 4

Commit message: update
Parts:
- added C10: 100nf, Capacitor_SMD:C_0402_1005Metric_Pad0.74x0.62mm_HandSolder, F.Cu at (152.4, 76.3)
- added C11: 100nf, Capacitor_SMD:C_0402_1005Metric_Pad0.74x0.62mm_HandSolder, F.Cu at (150.7, 78.8)
- added C12: 0.1uF, Capacitor_SMD:C_0402_1005Metric, F.Cu at (162.5, 76.3)
- added C13: 1uF, Capacitor_SMD:C_0402_1005Metric, F.Cu at (159.6, 78.3)
- added C14: 100nF, Capacitor_SMD:C_0402_1005Metric, F.Cu at (164.2, 74.3)
- added C15: 100nf, Capacitor_SMD:C_0402_1005Metric_Pad0.74x0.62mm_HandSolder, F.Cu at (152.4, 74.3)
- added C16: 100nf, Capacitor_SMD:C_0402_1005Metric_Pad0.74x0.62mm_HandSolder, F.Cu at (147.5, 80.7)
- added C17: 1uF, Capacitor_SMD:C_0402_1005Metric, F.Cu at (159.3, 80.3)
- added C18: 100nf, Capacitor_SMD:C_0402_1005Metric_Pad0.74x0.62mm_HandSolder, F.Cu at (147.5, 78.8)
- added C19: 100nF, Capacitor_SMD:C_0402_1005Metric, F.Cu at (195.5, 78.4)
- added C20: 2.2uF, Capacitor_SMD:C_0402_1005Metric, F.Cu at (206.1, 70.6)
- added C21: 1uF, Capacitor_SMD:C_0402_1005Metric, F.Cu at (209.0, 68.6)
- added C22: 100nF, Capacitor_SMD:C_0402_1005Metric, F.Cu at (200.5, 73.1)
- added C23: 2.2uF, Capacitor_SMD:C_0402_1005Metric, F.Cu at (206.1, 68.6)
- added C24: 10uF, Capacitor_SMD:C_1206_3216Metric, F.Cu at (188.2, 69.3)
- added C25: 10uF, Capacitor_SMD:C_1206_3216Metric, F.Cu at (188.2, 72.7)
- added C26: 1uF, Capacitor_SMD:C_0402_1005Metric, F.Cu at (192.6, 80.4)
- added C27: 100nF, Capacitor_SMD:C_0402_1005Metric, F.Cu at (203.4, 72.6)
- added C28: 100nF, Capacitor_SMD:C_0402_1005Metric, F.Cu at (198.4, 77.0)
- added C29: 2.2uF, Capacitor_SMD:C_0402_1005Metric, F.Cu at (201.1, 75.0)
- added C30: 2.2uF, Capacitor_SMD:C_0402_1005Metric, F.Cu at (198.2, 75.0)
- added C31: 1uF, Capacitor_SMD:C_0402_1005Metric, F.Cu at (203.2, 70.6)
- added C32: 1uF, Capacitor_SMD:C_0402_1005Metric, F.Cu at (198.4, 79.0)
- added C33: 100nF, Capacitor_SMD:C_0402_1005Metric, F.Cu at (195.5, 80.4)
- added C34: 22uF, Capacitor_SMD:C_1206_3216Metric, F.Cu at (188.2, 76.0)
- added C35: 22uF, Capacitor_SMD:C_1206_3216Metric, F.Cu at (193.8, 69.3)
- added C9: 100pF, Capacitor_SMD:C_0402_1005Metric, F.Cu at (156.1, 82.7)
- added L1: 10uH, Inductor_SMD:L_Bourns-SRN4018, F.Cu at (208.3, 81.5)
- added Q2: MMBT3904, Package_TO_SOT_SMD:SOT-23, F.Cu at (148.3, 75.6)
- added R10: 10K/1%, Resistor_SMD:R_0402_1005Metric, F.Cu at (156.7, 76.3)
- added R11: 5.1K/1%, Resistor_SMD:R_0402_1005Metric, F.Cu at (155.4, 74.3)
- added R12: 5.1K/1%, Resistor_SMD:R_0402_1005Metric, F.Cu at (150.3, 82.7)
- added R13: 1K, Resistor_SMD:R_0402_1005Metric, F.Cu at (150.6, 80.8)
- added R14: 10K/1%, Resistor_SMD:R_0402_1005Metric, F.Cu at (161.3, 74.3)
- added R15: 1K/1%, Resistor_SMD:R_0402_1005Metric, F.Cu at (153.8, 78.3)
- added R16: 10K, Resistor_SMD:R_0402_1005Metric, F.Cu at (147.3, 82.7)
- added R17: 1M, Resistor_SMD:R_0402_1005Metric, F.Cu at (195.4, 76.4)
- added R18: 100K, Resistor_SMD:R_0402_1005Metric, F.Cu at (197.6, 73.1)
- added R19: 560K, Resistor_SMD:R_0402_1005Metric, F.Cu at (189.7, 80.7)
- added R20: 51K, Resistor_SMD:R_0402_1005Metric, F.Cu at (186.8, 80.7)
- added R21: 20, Resistor_SMD:R_0402_1005Metric, F.Cu at (186.8, 78.7)
- added R22: 7.68K, Resistor_SMD:R_0402_1005Metric, F.Cu at (192.4, 76.4)
- added R23: 10K, Resistor_SMD:R_0402_1005Metric, F.Cu at (189.7, 78.7)
- added R24: 41.2K, Resistor_SMD:R_0402_1005Metric, F.Cu at (203.2, 68.6)
- added R25: 10K, Resistor_SMD:R_0402_1005Metric, F.Cu at (192.6, 78.4)
- added R4: 750K/0.1%, Resistor_SMD:R_0402_1005Metric, F.Cu at (158.4, 74.3)
- added R5: 2.37K/0.1%, Resistor_SMD:R_0402_1005Metric, F.Cu at (153.2, 82.7)
- added R6: 1K, Resistor_SMD:R_0402_1005Metric, F.Cu at (159.6, 76.3)
- added R7: 1K, Resistor_SMD:R_0402_1005Metric, F.Cu at (153.5, 80.8)
- added R8: 100K, Resistor_SMD:R_0402_1005Metric, F.Cu at (156.7, 78.3)
- added R9: 75K/1%, Resistor_SMD:R_0402_1005Metric, F.Cu at (156.4, 80.3)
- added U8: LP5907MFX-3.3, Package_TO_SOT_SMD:SOT-23-5, F.Cu at (199.2, 69.8)
- added U9: LP5907MFX-1.8, Package_TO_SOT_SMD:SOT-23-5, F.Cu at (193.6, 73.2)
- U3: value SGM8557 -> SGM8557-1AXN5G/TR
- U5: value CH224K -> CH340E; footprint kicad_lceda:ESSOP-10_L4.9-W3.9-P1.0-LS6.0-TL-EP -> Package_SO:MSOP-10_3x3mm_P0.5mm
- U7: value CH340E -> CH224K; footprint Package_SO:MSOP-10_3x3mm_P0.5mm -> kicad_lceda:ESSOP-10_L4.9-W3.9-P1.0-LS6.0-TL-EP
- moved J2 9.00 mm to (145.9, 92.4)
- moved J5 9.00 mm to (145.9, 92.4)
- moved J4 4.20 mm to (122.4, 92.5)
- moved J7 4.20 mm to (122.4, 92.5)
- moved J3 2.70 mm to (153.6, 92.4)
- moved J6 2.70 mm to (153.6, 92.4)
- moved C1 1.56 mm to (178.4, 84.4)
- moved C2 1.56 mm to (170.8, 72.0)
- moved C3 1.56 mm to (176.5, 71.9)
- moved C6 1.56 mm to (175.5, 84.4)
- moved C7 1.56 mm to (173.6, 72.0)
- moved D1 1.56 mm to (168.1, 70.0)
- moved R3 1.56 mm to (171.0, 70.0)
- moved C4 1.56 mm to (173.9, 70.0)
- moved C8 1.56 mm to (176.8, 70.0)
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Connections:
- net Net-(Q1-Pad5) renamed A
- CN1 pad 1: unconnected-(CN1-Pad1) -> Net-(CN1-Pad1)
- CN1 pad 10: unconnected-(CN1-Pad10) -> Net-(CN1-Pad10)
- CN1 pad 11: unconnected-(CN1-Pad11) -> Net-(CN1-Pad11)
- CN1 pad 12: unconnected-(CN1-Pad12) -> GND
- CN1 pad 13: unconnected-(CN1-Pad13) -> SDA
- CN1 pad 14: unconnected-(CN1-Pad14) -> SCL
- CN1 pad 15: unconnected-(CN1-Pad15) -> DCX
- CN1 pad 16: unconnected-(CN1-Pad16) -> RESET
- CN1 pad 17: unconnected-(CN1-Pad17) -> CS
- CN1 pad 19: unconnected-(CN1-Pad19) -> TP1
- CN1 pad 2: unconnected-(CN1-Pad2) -> Net-(CN1-Pad2)
- CN1 pad 20: unconnected-(CN1-Pad20) -> TP2
- CN1 pad 21: unconnected-(CN1-Pad21) -> TP3
- CN1 pad 22: unconnected-(CN1-Pad22) -> TP4
- CN1 pad 23: unconnected-(CN1-Pad23) -> TP5
- CN1 pad 24: unconnected-(CN1-Pad24) -> TP6
- CN1 pad 3: unconnected-(CN1-Pad3) -> Net-(CN1-Pad3)
- CN1 pad 4: unconnected-(CN1-Pad4) -> Net-(CN1-Pad4)
- CN1 pad 5: unconnected-(CN1-Pad5) -> +3V3
- CN1 pad 6: unconnected-(CN1-Pad6) -> GND
- CN1 pad 7: unconnected-(CN1-Pad7) -> +3V3
- CN1 pad 9: unconnected-(CN1-Pad9) -> Net-(CN1-Pad9)
- J1 pad A1: Net-(J1-PadA1) -> GND
- J1 pad A12: Net-(J1-PadA1) -> GND
- J1 pad A4: Net-(J1-PadA4) -> VBUS
- J1 pad A5: unconnected-(J1-PadA5) -> Net-(J1-PadA5)
- J1 pad A6: unconnected-(J1-PadA6) -> USB_DP
- J1 pad A7: unconnected-(J1-PadA7) -> USB_DM
- J1 pad A9: Net-(J1-PadA4) -> VBUS
- J1 pad B1: Net-(J1-PadA1) -> GND
- J1 pad B12: Net-(J1-PadA1) -> GND
- J1 pad B4: Net-(J1-PadA4) -> VBUS
- J1 pad B5: unconnected-(J1-PadB5) -> Net-(J1-PadB5)
- J1 pad B6: unconnected-(J1-PadB6) -> USB_DP
- J1 pad B7: unconnected-(J1-PadB7) -> USB_DM
- J1 pad B9: Net-(J1-PadA4) -> VBUS
- J1 pad S1: unconnected-(J1-PadS1) -> GND
- Q1 pad 1: Net-(Q1-Pad1) -> VBUS
- Q1 pad 2: Net-(Q1-Pad1) -> VBUS
- Q1 pad 3: Net-(Q1-Pad1) -> VBUS
- Q1 pad 4: unconnected-(Q1-Pad4) -> Net-(Q1-Pad4)
- U1 pad 10: EN1 -> unconnected-(U1-Pad10)
- U1 pad 12: USART2_TX -> unconnected-(U1-Pad12)
- U1 pad 13: USART2_RX -> unconnected-(U1-Pad13)
- U1 pad 18: Button -> unconnected-(U1-Pad18)
- U1 pad 22: ERROR -> unconnected-(U1-Pad22)
- U1 pad 25: SPI2_CS -> unconnected-(U1-Pad25)
- U1 pad 26: SPI2_SCK -> CFG1
- U1 pad 27: SPI2_MISO -> CFG2
- U1 pad 28: SPI2_MOSI -> CFG3
- U1 pad 29: PWMA -> unconnected-(U1-Pad29)
- U1 pad 30: PWMB -> USART_RX
- U1 pad 31: PWMC -> USART_TX
- U1 pad 32: USB_DM -> unconnected-(U1-Pad32)
- U1 pad 33: USB_DP -> unconnected-(U1-Pad33)
- U1 pad 42: I2C1_SCL -> SCL
- U1 pad 43: I2C1_SDA -> SDA
- U2 pad 1: unconnected-(U2-Pad1) -> SCK
- U2 pad 10: unconnected-(U2-Pad10) -> +1V8
- U2 pad 2: unconnected-(U2-Pad2) -> CS
- U2 pad 3: unconnected-(U2-Pad3) -> SD0
- U2 pad 4: unconnected-(U2-Pad4) -> SDA
- U2 pad 5: unconnected-(U2-Pad5) -> GND
- U2 pad 6: unconnected-(U2-Pad6) -> GND
- U2 pad 7: unconnected-(U2-Pad7) -> GND
- U2 pad 8: unconnected-(U2-Pad8) -> GND
- U2 pad 9: unconnected-(U2-Pad9) -> +1V8
- U3 pad 1: unconnected-(U3-Pad1) -> Net-(C9-Pad1)
- U3 pad 2: unconnected-(U3-Pad2) -> B
- U3 pad 3: unconnected-(U3-Pad3) -> Net-(R8-Pad1)
- U3 pad 4: (no net) -> Net-(C9-Pad2)
- U3 pad 5: (no net) -> +5V
- U4 pad 1: unconnected-(U4-Pad1) -> Net-(U4-Pad1)
- U4 pad 2: unconnected-(U4-Pad2) -> +5V
- U4 pad 4: unconnected-(U4-Pad4) -> +5V
- U4 pad 5: unconnected-(U4-Pad5) -> GND
- U5 pad 1: unconnected-(U5-Pad1) -> USB_DP
- U5 pad 10: unconnected-(U5-Pad10) -> +3V3
- U5 pad 2: unconnected-(U5-Pad2) -> USB_DM
- U5 pad 3: unconnected-(U5-Pad3) -> GND
- U5 pad 7: unconnected-(U5-Pad7) -> +3V3
- U5 pad 8: unconnected-(U5-Pad8) -> USART_RX
- U5 pad 9: unconnected-(U5-Pad9) -> USART_TX
- U6 pad 1: unconnected-(U6-Pad1) -> Net-(U6-Pad1)
- U6 pad 2: unconnected-(U6-Pad2) -> VBUS
- U6 pad 3: unconnected-(U6-Pad3) -> Net-(U6-Pad3)
- U6 pad 4: unconnected-(U6-Pad4) -> GND
- U6 pad 5: unconnected-(U6-Pad5) -> Net-(U6-Pad5)
- U6 pad 6: unconnected-(U6-Pad6) -> Net-(U6-Pad6)
- U6 pad 7: unconnected-(U6-Pad7) -> Net-(U6-Pad7)
- U6 pad 8: unconnected-(U6-Pad8) -> Net-(U6-Pad8)
- U7 pad 1: unconnected-(U7-Pad1) -> Net-(C17-Pad1)
- U7 pad 2: unconnected-(U7-Pad2) -> CFG2
- U7 pad 3: unconnected-(U7-Pad3) -> CFG3
- U7 pad 4: unconnected-(U7-Pad4) -> USB_DP
- U7 pad 5: unconnected-(U7-Pad5) -> USB_DM
- U7 pad 6: unconnected-(U7-Pad6) -> Net-(J1-PadB5)
- U7 pad 7: unconnected-(U7-Pad7) -> Net-(J1-PadA5)
- U7 pad 8: unconnected-(U7-Pad8) -> Net-(R16-Pad1)
- U7 pad 9: unconnected-(U7-Pad9) -> CFG1
Other:
- board size 100 x 13 mm -> 95.8 x 13 mm

Commit message: update
Parts:
- added R26: 10K/1%, Resistor_SMD:R_0402_1005Metric, F.Cu at (193.0, 105.7)
- added R27: 10K/1%, Resistor_SMD:R_0402_1005Metric, F.Cu at (190.1, 105.7)
- added SW1: SW_Push, Button_Switch_SMD:SW_SPST_PTS810, F.Cu at (159.2, 92.4)
- added SW2: SW_Push, Button_Switch_SMD:SW_SPST_PTS810, F.Cu at (174.4, 92.7)
- C12, C24, C25, C27, C28, C33, C34, C35, C9, L1, Q1, R17, R18, R20, R21, R22, R24, R4, R5, R6, R8, U3: moved to B.Cu
- J2: value Conn_01x04 -> Negative
- J3: value Conn_01x04 -> Positive
- J7: value Conn_01x04 -> Com
- moved R24 90.0 mm to (113.5, 75.2), turned to 180 degrees
- moved C27 89.2 mm to (114.2, 69.9), turned to 180 degrees
- moved C28 84.5 mm to (114.0, 72.4), turned to 180 degrees
- moved L1 79.3 mm to (130.0, 68.9), turned to 180 degrees
- moved C25 74.1 mm to (114.3, 67.7), turned to 180 degrees
- moved C24 74.1 mm to (114.3, 64.7), turned to 180 degrees
- moved C33 72.1 mm to (125.5, 63.1), turned to 180 degrees
- moved U6 71.9 mm to (124.0, 67.7)
- moved R21 71.7 mm to (117.2, 61.1), turned to 180 degrees
- moved R17 71.4 mm to (124.1, 71.9), turned to 180 degrees
- moved R18 70.1 mm to (127.5, 74.4), turned to 180 degrees
- moved R20 66.9 mm to (120.0, 75.9), turned to 180 degrees
- moved R22 64.7 mm to (127.8, 76.4), turned to 180 degrees
- moved C35 55.4 mm to (138.5, 72.2), turned to 180 degrees
- moved C34 49.5 mm to (139.2, 68.7), turned to 180 degrees
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Connections:
- C15 pad 1: Net-(C15-Pad1) -> Vin_Sense
- CN1 pad 25: unconnected-(CN1-Pad25) -> GND
- CN1 pad 26: unconnected-(CN1-Pad26) -> GND
- CN1 pad 27: unconnected-(CN1-Pad27) -> GND
- CN1 pad 28: unconnected-(CN1-Pad28) -> GND
- J2 pad 1: unconnected-(J2-Pad1) -> B
- J2 pad 2: unconnected-(J2-Pad2) -> B
- J2 pad 3: unconnected-(J2-Pad3) -> B
- J2 pad 4: unconnected-(J2-Pad4) -> B
- J3 pad 1: unconnected-(J3-Pad1) -> A
- J3 pad 2: unconnected-(J3-Pad2) -> A
- J3 pad 3: unconnected-(J3-Pad3) -> A
- J3 pad 4: unconnected-(J3-Pad4) -> A
- J4 pad 1: unconnected-(J4-Pad1) -> GND
- J4 pad 2: unconnected-(J4-Pad2) -> GND
- J4 pad 3: unconnected-(J4-Pad3) -> GND
- J4 pad 4: unconnected-(J4-Pad4) -> GND
- J5 pad 1: unconnected-(J5-Pad1) -> B
- J5 pad 2: unconnected-(J5-Pad2) -> B
- J5 pad 3: unconnected-(J5-Pad3) -> B
- J5 pad 4: unconnected-(J5-Pad4) -> B
- J6 pad 1: unconnected-(J6-Pad1) -> A
- J6 pad 2: unconnected-(J6-Pad2) -> A
- J6 pad 3: unconnected-(J6-Pad3) -> A
- J6 pad 4: unconnected-(J6-Pad4) -> A
- J7 pad 1: unconnected-(J7-Pad1) -> GND
- J7 pad 2: unconnected-(J7-Pad2) -> GND
- J7 pad 3: unconnected-(J7-Pad3) -> GND
- J7 pad 4: unconnected-(J7-Pad4) -> GND
- R10 pad 1: Net-(C15-Pad1) -> Vin_Sense
- R9 pad 2: Net-(C15-Pad1) -> Vin_Sense
- U1 pad 10: unconnected-(U1-Pad10) -> Vin_Sense
- U1 pad 11: unconnected-(U1-Pad11) -> Tip_Temp
- U1 pad 12: unconnected-(U1-Pad12) -> Board_Temp
- U1 pad 13: unconnected-(U1-Pad13) -> Tip_Control
- U1 pad 22: unconnected-(U1-Pad22) -> Button1
- U1 pad 25: unconnected-(U1-Pad25) -> Button2
- U1 pad 32: unconnected-(U1-Pad32) -> INT1
- U1 pad 33: unconnected-(U1-Pad33) -> INT2
- U2 pad 11: unconnected-(U2-Pad11) -> INT2
- U2 pad 12: unconnected-(U2-Pad12) -> INT1
Other:
- board size 95.8 x 13 mm -> 100 x 13 mm

Commit message: update
Parts:
- removed C1, C4: 30PF, Capacitor_SMD:C_0402_1005Metric
- C10, C11, C15, C16, C17, C18, Q2, R10, R11, R12, R13, R14, R15, R16, R9: moved to B.Cu
- moved C24 82.0 mm to (189.2, 97.8), turned to 0 degrees
- moved C25 79.9 mm to (189.2, 95.3), turned to 0 degrees
- moved R24 79.4 mm to (192.0, 87.2), turned to 90 degrees
- moved C27 78.8 mm to (189.5, 93.3), turned to 0 degrees
- moved C28 77.1 mm to (189.6, 87.3), turned to 0 degrees
- moved R21 74.6 mm to (187.2, 87.0)
- moved R20 73.2 mm to (192.0, 89.2), turned to 90 degrees
- moved R17 71.4 mm to (192.2, 93.2), turned to 0 degrees
- moved U6 69.6 mm to (189.8, 90.5)
- moved C33 67.3 mm to (187.8, 88.8), turned to -90 degrees
- moved R18 66.9 mm to (192.2, 91.7), turned to 0 degrees
- moved R22 66.7 mm to (193.2, 89.2), turned to -90 degrees
- moved L1 59.2 mm to (184.8, 91.5), turned to -90 degrees
- moved R13 57.7 mm to (207.8, 88.8), turned to 180 degrees
- moved C35 52.1 mm to (183.9, 97.8)
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Routing:
- net Net-(J1-PadA5): track 0.00 -> 16.9 mm
- net +5V: track 0.00 -> 14.2 mm, vias 0 -> 2
- net Net-(J1-PadB5): track 0.00 -> 13.2 mm
- net +3V3: track 0.00 -> 12.6 mm
- net VBUS: track 0.00 -> 11.1 mm
- net Net-(C28-Pad2): track 0.00 -> 10.7 mm, vias 0 -> 2
- net Net-(R17-Pad2): track 0.00 -> 9.94 mm, vias 0 -> 2
- net Net-(C6-Pad1): track 0.00 -> 9.47 mm, vias 0 -> 2
- net GND: track 0.00 -> 8.61 mm, vias 0 -> 9
- net USB_DM: track 0.00 -> 4.79 mm, vias 0 -> 1
- net USB_DP: track 0.00 -> 4.39 mm, vias 0 -> 1
- net Net-(C17-Pad1): track 0.00 -> 4.02 mm
- net HSE_IN: track 0.00 -> 3.41 mm
- net HSE_OUT: track 0.00 -> 2.93 mm
- net Net-(D1-Pad2): track 0.00 -> 2.40 mm
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- added copper zone on B.Cu, net +5V
- added copper zone on B.Cu, net GND
- added copper zone on B.Cu, net Net-(L1-Pad1)
- added copper zone on B.Cu, net VBUS

Commit message: PCB layout update
Parts:
- added C1: 1uF, Capacitor_SMD:C_0402_1005Metric, F.Cu at (168.5, 90.3)
- added J8: Conn_01x04, Connector_JST:JST_SH_BM04B-SRSS-TB_1x04-1MP_P1.00mm_Vertical, F.Cu at (196.6, 96.3)
- added R28: 1K, Resistor_SMD:R_0402_1005Metric, F.Cu at (202.0, 96.4)
- added R29: 1K, Resistor_SMD:R_0402_1005Metric, F.Cu at (202.1, 98.2)
- C19, C20, C21, C23, U8: moved to B.Cu
- moved C23 16.7 mm to (186.1, 88.6), turned to 0 degrees
- moved U5 16.3 mm to (180.4, 91.9)
- moved C21 15.3 mm to (186.1, 90.0), turned to 0 degrees
- moved C11 14.7 mm to (181.6, 95.7)
- moved C10 14.6 mm to (181.6, 97.0)
- moved U8 11.0 mm to (185.6, 92.8), turned to 90 degrees
- moved R25 9.77 mm to (209.8, 91.2), turned to 180 degrees
- moved R16 9.67 mm to (206.1, 97.8), turned to 0 degrees
- moved U9 9.44 mm to (169.3, 88.1), turned to 180 degrees
- moved C30 9.31 mm to (202.7, 92.6)
- moved C29 9.30 mm to (202.7, 91.4)
- moved R19 9.27 mm to (202.8, 90.3)
- moved R24 9.10 mm to (201.1, 87.2), turned to 180 degrees
- moved R17 8.58 mm to (200.8, 92.9)
- moved R18 8.58 mm to (200.8, 91.4)
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Connections:
- CN1 pad 17: CS -> DISPLAY_CS
- U1 pad 14: CS -> DISPLAY_CS
- U1 pad 15: SCK -> SCL
- U1 pad 16: MISO -> RESET
- U1 pad 17: MOSI -> SDA
- U1 pad 18: unconnected-(U1-Pad18) -> Voltage
- U1 pad 21: unconnected-(U1-Pad21) -> CFG2
- U1 pad 22: Button1 -> CFG3
- U1 pad 25: Button2 -> IMU_CS
- U1 pad 26: CFG1 -> IMU_SCK
- U1 pad 27: CFG2 -> IMU_SD0
- U1 pad 28: CFG3 -> IMU_SDA
- U1 pad 29: unconnected-(U1-Pad29) -> DCX
- U1 pad 32: INT1 -> USB_DP
- U1 pad 33: INT2 -> USB_DM
- U1 pad 41: unconnected-(U1-Pad41) -> INT2
- U1 pad 42: SCL -> INT1
- U1 pad 43: SDA -> Button1
- U1 pad 45: unconnected-(U1-Pad45) -> Button2
- U1 pad 46: unconnected-(U1-Pad46) -> CFG1
- U2 pad 1: SCK -> IMU_SCK
- U2 pad 2: CS -> IMU_CS
- U2 pad 3: SD0 -> IMU_SD0
- U2 pad 4: SDA -> IMU_SDA
Routing:
- net USB_DP: track 4.39 -> 56.7 mm, vias 1 -> 2
- net USB_DM: track 4.79 -> 50.2 mm, vias 1 -> 2
- net INT2: track 0.00 -> 43.7 mm, vias 0 -> 2
- net CFG3: track 0.00 -> 39.9 mm, vias 0 -> 2
- net IMU_SCK: track 0.00 -> 39.3 mm, vias 0 -> 2
- net INT1: track 0.00 -> 38.8 mm, vias 0 -> 2
- net Button1: track 0.00 -> 35.1 mm, vias 0 -> 2
- net DISPLAY_CS: track 0.00 -> 34.3 mm, vias 0 -> 2
- net RESET: track 0.00 -> 34.0 mm, vias 0 -> 2
- net +3V3: track 12.6 -> 45.3 mm, vias 0 -> 1
- net SCL: track 0.00 -> 32.1 mm, vias 0 -> 2
- net SDA: track 0.00 -> 31.8 mm, vias 0 -> 2
- net GND: track 8.61 -> 40.0 mm, vias 9 -> 11
- net CFG1: track 0.00 -> 30.2 mm, vias 0 -> 3
- net Tip_Control: track 0.00 -> 28.9 mm, vias 0 -> 1
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- added copper zone on B.Cu, net A
- added copper zone on F.Cu, net A
- added copper zone on F.Cu, net GND
- added copper zone on In1.Cu, net GND
- added copper zone on In2.Cu, net GND

Commit message: PCB layout update
Parts:
- R28: value 1K -> 50K
- R29: value 1K -> 9K
- moved C7 0.41 mm to (188.7, 98.0)
- moved JP1 0.09 mm to (190.1, 87.0)
Connections:
- U1 pad 32: USB_DP -> unconnected-(U1-Pad32)
- U1 pad 33: USB_DM -> unconnected-(U1-Pad33)
Routing:
- net +3V3: track 45.3 -> 95.9 mm, vias 1 -> 15
- net B: track 0.00 -> 38.1 mm, vias 0 -> 3
- net Vin_Sense: track 4.48 -> 23.4 mm, vias 1 -> 2
- net +5V: track 21.4 -> 40.0 mm, vias 3 -> 12
- net A: track 1.26 -> 19.1 mm, vias 75 -> 45
- net GND: track 40.0 -> 55.1 mm, vias 11 -> 55
- net Tip_Temp: track 1.41 -> 15.8 mm, vias 1 -> 2
- net VBUS: track 30.1 -> 35.3 mm, vias 0 -> 14
- net IMU_SCK: track 39.3 -> 34.3 mm
- net USB_DM: track 50.2 -> 46.1 mm
- net USB_DP: track 56.7 -> 53.8 mm
- net Net-(C28-Pad2): track 9.92 -> 8.96 mm
- net INT1: track 38.8 -> 39.7 mm
- net RESET: track 34.0 -> 33.5 mm
- added copper zone on B.Cu, net +3V3
- added copper zone on In1.Cu, net +3V3
- added copper zone on In2.Cu, net +5V
- added copper zone on B.Cu, net B
- added copper zone on F.Cu, net B
- added copper zone on In1.Cu, net VBUS

Commit message: PCB layout update
Parts:
- added C36: 100nF, Capacitor_SMD:C_0402_1005Metric, F.Cu at (167.2, 95.2)
- added C37: 100nF, Capacitor_SMD:C_0402_1005Metric, F.Cu at (169.4, 95.2)
- added C4: 1uf, Capacitor_SMD:C_0402_1005Metric, F.Cu at (171.2, 92.2)
- added R30: 10K/1%, Resistor_SMD:R_0402_1005Metric, F.Cu at (164.9, 97.8)
- added R31: 10K/1%, Resistor_SMD:R_0402_1005Metric, F.Cu at (171.6, 97.8)
- added R32: 10K/1%, Resistor_SMD:R_0402_1005Metric, F.Cu at (168.8, 89.5)
- added R33: 10K/1%, Resistor_SMD:R_0402_1005Metric, F.Cu at (167.8, 89.5)
- added R34: 10K/1%, Resistor_SMD:R_0402_1005Metric, F.Cu at (166.8, 89.5)
- added R35: 10K/1%, Resistor_SMD:R_0402_1005Metric, F.Cu at (165.0, 96.2)
- added R36: 10K/1%, Resistor_SMD:R_0402_1005Metric, F.Cu at (171.6, 96.2)
- added U10: TXS0102DCU, Package_SO:VSSOP-8_2.3x2mm_P0.5mm, F.Cu at (168.3, 97.1)
- moved U9 2.17 mm to (171.4, 88.0)
- moved C1 2.17 mm to (170.6, 90.2)
- moved C22 0.85 mm to (170.2, 92.1)
- moved U2 0.85 mm to (168.2, 92.4)
- moved R26 0.28 mm to (158.7, 96.3)
Connections:
- U1 pad 18: Voltage -> unconnected-(U1-Pad18)
- U1 pad 21: CFG2 -> IMU_SCL_3.3V
- U1 pad 22: CFG3 -> IMU_SDA_3.3V
- U1 pad 25: IMU_CS -> unconnected-(U1-Pad25)
- U1 pad 26: IMU_SCK -> unconnected-(U1-Pad26)
- U1 pad 27: IMU_SD0 -> unconnected-(U1-Pad27)
- U1 pad 28: IMU_SDA -> unconnected-(U1-Pad28)
- U1 pad 3: unconnected-(U1-Pad3) -> Button2
- U1 pad 4: unconnected-(U1-Pad4) -> Button1
- U1 pad 41: INT2 -> CFG1
- U1 pad 42: INT1 -> CFG2
- U1 pad 43: Button1 -> CFG3
- U1 pad 45: Button2 -> INT1
- U1 pad 46: CFG1 -> INT2
- U2 pad 1: IMU_SCK -> IMU_SCL_1.8V
- U2 pad 3: IMU_SD0 -> IMU_SD0_1.8V
- U2 pad 4: IMU_SDA -> IMU_SDA_1.8V
Routing:
- net IMU_SCK: track 34.3 -> 0.00 mm, vias 2 -> 0
- net +1V8: track 7.93 -> 36.2 mm, vias 0 -> 2
- net INT2: track 43.8 -> 17.8 mm
- net IMU_SDA_3.3V: track 0.00 -> 25.4 mm, vias 0 -> 2
- net IMU_SD0: track 24.2 -> 0.00 mm, vias 2 -> 0
- net IMU_CS: track 26.3 -> 2.58 mm, vias 2 -> 0
- net IMU_SDA: track 22.0 -> 0.00 mm, vias 2 -> 0
- net IMU_SCL_3.3V: track 0.00 -> 20.8 mm, vias 0 -> 2
- net INT1: track 39.7 -> 19.6 mm
- net Voltage: track 20.6 -> 1.72 mm
- net +3V3: track 95.9 -> 114.3 mm, vias 15 -> 16
- net IMU_SCL_1.8V: track 0.00 -> 15.3 mm, vias 0 -> 2
- net CFG3: track 39.4 -> 26.7 mm
- net IMU_SDA_1.8V: track 0.00 -> 9.81 mm, vias 0 -> 2
- net Button1: track 35.3 -> 31.2 mm
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Other:
- board size 100 x 13 mm -> 100 x 13.8 mm
