File: Mini_Solder_Iron/Mini_Solder_Iron.kicad_pcb (KiCad board)
At the start: 4 copper layers, 100 x 13.8 mm, 100 parts, among them CN1 YXT-BB10-24S-02, J1 USB_C_Receptacle_USB2.0, J2 Negative, J3 Positive, J4 Conn_01x04, J5 Conn_01x04, J6 Conn_01x04, J7 Com, J8 Conn_01x04, Q1 AO4407A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

Commit message: PCB layout update
Parts:
- removed C10, C11: 100nf, Capacitor_SMD:C_0402_1005Metric_Pad0.74x0.62mm_HandSolder
- removed R28: 50K, Resistor_SMD:R_0402_1005Metric
- removed R29: 9K, Resistor_SMD:R_0402_1005Metric
- removed U5: CH340E, Package_SO:MSOP-10_3x3mm_P0.5mm
- J8: value Conn_01x04 -> Conn_01x06; footprint Connector_JST:JST_SH_BM04B-SRSS-TB_1x04-1MP_P1.00mm_Vertical -> Connector_JST:JST_SH_BM06B-SRSS-TB_1x06-1MP_P1.00mm_Vertical
- moved C26 0.72 mm to (202.7, 94.5)
- moved C29 0.72 mm to (202.7, 92.2)
- moved C30 0.72 mm to (202.7, 93.3)
- moved C31 0.72 mm to (202.7, 88.3)
- moved C32 0.72 mm to (202.7, 89.6)
- moved CN1 0.72 mm to (206.2, 90.5)
- moved R19 0.72 mm to (202.8, 91.0)
- moved R23 0.72 mm to (209.8, 93.1)
- moved R25 0.72 mm to (209.8, 91.9)
- moved C7 0.53 mm to (189.2, 98.0)
- moved JP1 0.39 mm to (190.0, 86.6)
- moved C3 0.29 mm to (180.6, 88.0)
Connections:
- J8 pad 4: GND -> USART_TX
Routing:
- net USB_DP: track 54.5 -> 9.68 mm, vias 2 -> 0
- net USB_DM: track 46.4 -> 7.47 mm, vias 2 -> 0
- net VBUS: track 35.5 -> 29.8 mm
- net +3V3: track 114.3 -> 117.7 mm, vias 16 -> 15
- net Net-(R27-Pad2): track 8.50 -> 6.23 mm
- net USART_RX: track 9.98 -> 7.72 mm, vias 1 -> 0
- net CFG3: track 26.7 -> 28.7 mm
- net USART_TX: track 10.8 -> 8.98 mm, vias 1 -> 0
- net Voltage: track 1.72 -> 0.00 mm
- net DCX: track 26.3 -> 24.8 mm
- net SCL: track 31.7 -> 30.7 mm
- net GND: track 57.1 -> 56.3 mm, vias 54 -> 55
- net SDA: track 31.4 -> 30.7 mm
- net CFG1: track 29.0 -> 28.4 mm
- net RESET: track 33.5 -> 32.9 mm
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
Commit message: PCB layout update
Parts:
- moved JP1 0.40 mm to (190.2, 87.0)
- moved R18 0.38 mm to (201.2, 91.5)
- moved C2 0.20 mm to (178.5, 94.3)
- moved R3 0.15 mm to (178.5, 95.5)
Routing:
- net +1V8: track 36.2 -> 33.0 mm
- net B: track 38.1 -> 40.6 mm, vias 3 -> 5
- net DISPLAY_CS: track 33.8 -> 32.7 mm
- net Net-(C28-Pad2): track 8.96 -> 8.08 mm
- net +3V3: track 117.7 -> 117.0 mm
Other:
- board size 100 x 13.8 mm -> 100 x 12.8 mm
- board text added: "Mini Solder iron"
- board text added: "V1.0"
