File: Mini_Solder_Iron/Mini_Solder_Iron.kicad_sch (KiCad schematic)
At the start: 9 parts, among them CN1 YXT-BB10-24S-02, J1 USB_C_Receptacle_USB2.0, Q1 AO4407A, U1 STM32F103C8Tx, U2 LIS2DS12, U3 SGM8557, U4 TMP36GRTZ, U5 CH224K, U6 MP9942

Commit message: update
Parts:
- removed U5: CH224K, kicad_lceda:ESSOP-10_L4.9-W3.9-P1.0-LS6.0-TL-EP, symbol kicad_lceda:CH224K
- added C1, C4: 30PF, Capacitor_SMD:C_0402_1005Metric, symbol Device:C_Small
- added C2: 4u7, Capacitor_SMD:C_0402_1005Metric, symbol Device:C_Small
- added C3, C5, C6, C7, C8: 100nf, Capacitor_SMD:C_0402_1005Metric, symbol Device:C_Small
- added C? (x2): 100nf, Capacitor_SMD:C_0402_1005Metric_Pad0.74x0.62mm_HandSolder, symbol Device:C_Small
- added D1: LED, LED_SMD:LED_0402_1005Metric, symbol Device:LED
- added J2, J5: Conn_01x04, kicad_lceda:JBC245_2.4mm, symbol Connector_Generic:Conn_01x04
- added J3, J6: Conn_01x04, kicad_lceda:JBC245_1.5mm, symbol Connector_Generic:Conn_01x04
- added J4, J7: Conn_01x04, kicad_lceda:JBC245_3.5mm, symbol Connector_Generic:Conn_01x04
- added JP1: SolderJumper_2_Open, Jumper:SolderJumper-2_P1.3mm_Open_RoundedPad1.0x1.5mm, symbol Jumper:SolderJumper_2_Open
- added R1, R3: 10K, Resistor_SMD:R_0402_1005Metric, symbol Device:R_Small
- added R2: 1K5, Resistor_SMD:R_0402_1005Metric, symbol Device:R_Small
- added U7, U?: CH340E, Package_SO:MSOP-10_3x3mm_P0.5mm, symbol Interface_USB:CH340E
- added Y1: Crystal_GND3_Small, CSTCE8M00G55:OSC_CSTCE8M00G55-R0, symbol Device:Crystal_GND3_Small
- U1: value STM32F103C8Tx -> STM32F103C8T6
Connections:
- net +3V3: now reaches U1.1 (VBAT)
- net +3V3: now also U1.24 (VDD), U1.36 (VDD), U1.48 (VDD), U1.9 (VDDA), C2.1, C3.1, C5.1, C7.1, C8.1, C?.1, C?.1, JP1.1 (A), R3.1, U?.10 (V3), U?.7 (VCC)
- net EN1: now reaches U1.10 (PA0)
- net USART2_TX: now reaches U1.12 (PA2)
- net USART2_RX: now reaches U1.13 (PA3)
- net CS: now reaches U1.14 (PA4)
- net SCK: now reaches U1.15 (PA5)
- net MISO: now reaches U1.16 (PA6)
- net MOSI: now reaches U1.17 (PA7)
- net Button: now reaches U1.18 (PB0)
- net at U1.2 (PC13): now also D1.2 (A)
- net ERROR: now reaches U1.22 (PB11)
- net GND: now reaches U1.23 (VSS)
- net GND: now also U1.35 (VSS), U1.47 (VSS), U1.8 (VSSA), C1.2, C2.2, C3.2, C4.2, C5.2, C6.2, C7.2, C8.2, C?.2, C?.2, R1.2, R2.2, U?.3 (GND), Y1.3
- net SPI2_CS: now reaches U1.25 (PB12)
- net SPI2_SCK: now reaches U1.26 (PB13)
- net SPI2_MISO: now reaches U1.27 (PB14)
- net SPI2_MOSI: now reaches U1.28 (PB15)
- net PWMA: now reaches U1.29 (PA8)
- net USART_RX: now reaches U1.30 (PA9)
- net USART_RX: now also U?.8 (TXD)
- net USART_TX: now reaches U1.31 (PA10)
- net USART_TX: now also U?.9 (RXD)
- net USB_DM: now reaches U1.32 (PA11)
- net USB_DP: now reaches U1.33 (PA12)
- net SWDIO: now reaches U1.34 (PA13)
- net SWCLK: now reaches U1.37 (PA14)
- net I2C1_SCL: now reaches U1.42 (PB6)
- net I2C1_SDA: now reaches U1.43 (PB7)
- net at U1.44 (BOOT0): now also JP1.2 (B), R1.1
- net HSE_IN: now reaches U1.5 (PD0)
- net HSE_IN: now also C4.1, Y1.2
- net HSE_OUT: now reaches U1.6 (PD1)
- net HSE_OUT: now also C1.1, Y1.1
- net at U1.7 (NRST): now also C6.1, R3.2
- new net: D1.1 (K), R2.1
- new net D+: U?.1 (UD+)
- new net D-: U?.2 (UD-)
- no-connect marks 0 -> 15
Other:
- note added: "STM32F103"
- moved on the sheet: CN1, J1, Q1, U2, U3A, U4, U6

Commit message: update
Parts:
- removed U3: SGM8557, Package_TO_SOT_SMD:SOT-23-5, symbol Amplifier_Operational:OPA2333xxD
- removed U7: CH340E, Package_SO:MSOP-10_3x3mm_P0.5mm, symbol Interface_USB:CH340E
- added C12: 0.1uF, Capacitor_SMD:C_0402_1005Metric, symbol Device:C_Small
- added C13, C17, C21, C26, C31, C32: 1uF, Capacitor_SMD:C_0402_1005Metric, symbol Device:C_Small
- added C14, C19, C22, C27, C28, C33: 100nF, Capacitor_SMD:C_0402_1005Metric, symbol Device:C_Small
- added C15, C16, C18: 100nf, Capacitor_SMD:C_0402_1005Metric_Pad0.74x0.62mm_HandSolder, symbol Device:C_Small
- added C20, C23, C29, C30: 2.2uF, Capacitor_SMD:C_0402_1005Metric, symbol Device:C_Small
- added C24, C25: 10uF, Capacitor_SMD:C_1206_3216Metric, symbol Device:C_Small
- added C34, C35: 22uF, Capacitor_SMD:C_1206_3216Metric, symbol Device:C_Small
- added C9: 100pF, Capacitor_SMD:C_0402_1005Metric, symbol Device:C_Small
- added L1: 10uH, Inductor_SMD:L_Bourns-SRN4018, symbol Device:L_Small
- added Q2: MMBT3904, Package_TO_SOT_SMD:SOT-23, symbol Transistor_BJT:MMBT3904
- added R10, R14: 10K/1%, Resistor_SMD:R_0402_1005Metric, symbol Device:R_Small
- added R11, R12: 5.1K/1%, Resistor_SMD:R_0402_1005Metric, symbol Device:R_Small
- added R13, R6, R7: 1K, Resistor_SMD:R_0402_1005Metric, symbol Device:R_Small
- added R15: 1K/1%, Resistor_SMD:R_0402_1005Metric, symbol Device:R_Small
- added R16, R23, R25: 10K, Resistor_SMD:R_0402_1005Metric, symbol Device:R_Small
- added R17: 1M, Resistor_SMD:R_0402_1005Metric, symbol Device:R_Small
- added R18, R8: 100K, Resistor_SMD:R_0402_1005Metric, symbol Device:R_Small
- added R19: 560K, Resistor_SMD:R_0402_1005Metric, symbol Device:R_Small
- added R20: 51K, Resistor_SMD:R_0402_1005Metric, symbol Device:R_Small
- added R21: 20, Resistor_SMD:R_0402_1005Metric, symbol Device:R_Small
- added R22: 7.68K, Resistor_SMD:R_0402_1005Metric, symbol Device:R_Small
- added R24: 41.2K, Resistor_SMD:R_0402_1005Metric, symbol Device:R_Small
- added R4: 750K/0.1%, Resistor_SMD:R_0402_1005Metric, symbol Device:R_Small
- added R5: 2.37K/0.1%, Resistor_SMD:R_0402_1005Metric, symbol Device:R_Small
- added R9: 75K/1%, Resistor_SMD:R_0402_1005Metric, symbol Device:R_Small
- added U3: SGM8557-1AXN5G/TR, Package_TO_SOT_SMD:SOT-23-5, symbol Amplifier_Operational:OPA340NA
- added U7: CH224K, kicad_lceda:ESSOP-10_L4.9-W3.9-P1.0-LS6.0-TL-EP, symbol kicad_lceda:CH224K
- added U8: LP5907MFX-3.3, Package_TO_SOT_SMD:SOT-23-5, symbol Regulator_Linear:LP5907MFX-3.3
- added U9: LP5907MFX-1.8, Package_TO_SOT_SMD:SOT-23-5, symbol Regulator_Linear:LP5907MFX-1.8
- gave numbers to parts that had none: 3
Connections:
- net D+ is gone; now on net USB_DP: U5.1 (UD+)
- net D- is gone; now on net USB_DM: U5.2 (UD-)
- net I2C1_SCL is gone; now on net SCL: U1.42 (PB6)
- net I2C1_SDA is gone; now on net SDA: U1.43 (PB7)
- net +3V3: now also CN1.5, CN1.7, C21.2, C23.2, C26.2, R23.1, R25.1, U8.5 (OUT), U9.1 (IN), U9.3 (EN)
- net CS: now also CN1.17, U2.2 (~{CS})
- net GND: now also CN1.12, CN1.6, J1.A1 (GND), J1.A12 (GND), J1.B1 (GND), J1.B12 (GND), J1.S1 (SHIELD), U2.5 (RES), U2.6 (GND), U2.7 (GND), U2.8 (GND), U4.5 (GND), U6.4 (GND), C13.2, C14.2, C15.2, C16.2, C17.2, C19.1, C20.1, C21.1, C22.1, C23.1, C24.1, C25.1, C26.1, C27.1, C28.1, C29.1, C30.1, C34.1, C35.1, Q2.2 (E), R10.2, R15.2, R19.1, R22.2, U7.0 (GND), U8.2 (GND), U9.2 (GND)
- net SCK: now also U2.1 (SCL/SPC)
- net USB_DM: now also J1.A7 (D-), J1.B7 (D-), U7.5 (DM); no longer U1.32 (PA11)
- net USB_DP: now also J1.A6 (D+), J1.B6 (D+), U7.4 (DP); no longer U1.33 (PA12)
- net at U6.1 (PG): now also R18.1
- net VBUS: now reaches U6.2 (IN)
- net VBUS: now also J1.A4 (VBUS), J1.A9 (VBUS), J1.B4 (VBUS), J1.B9 (VBUS), Q1.1, Q1.2, Q1.3, C24.2, C25.2, C27.2, R11.1, R13.1, R16.2, R17.1, R9.1
- net at U6.3 (SW): now also L1.1, R21.2
- net at U6.5 (BST): now also C33.2
- net at U6.6 (EN/SYNC): now also R17.2
- net at U6.7 (VCC): now also C28.2, R18.2
- net at U6.8 (FB): now also R20.1
- net at U4.1 (VOUT): now also R7.1
- net +5V: now reaches U4.2 (+VS)
- net +5V: now also U4.4 (~{SHUTDOWN}), C13.1, C14.1, C19.2, C20.2, C34.2, C35.2, L1.2, R24.2, U3.5 (V+), U8.1 (IN), U8.3 (EN)
- net at Q1.4: now also R11.2, R12.1
- net A: now reaches Q1.5, Q1.6, Q1.7, Q1.8
- net A: now also C12.2, R8.2
- net +1V8: now reaches U2.10 (Vdd_IO)
- net +1V8: now also U2.9 (Vdd), C22.2, U9.5 (OUT)
- net SD0: now reaches U2.3 (SA0/SDO)
- net SDA: now reaches U2.4 (SDA/SDI)
- net SDA: now also CN1.13, R23.2
- net at J1.A5 (CC1): now also U7.7 (CC1)
- net at J1.B5 (CC2): now also U7.6 (CC2)
- net at CN1.1: now also C31.2
- net at CN1.10: now also C29.2
- net at CN1.11: now also C30.2
- net SCL: now reaches CN1.14
- net SCL: now also R25.2
- net DCX: now reaches CN1.15
- net RESET: now reaches CN1.16
- net TP1: now reaches CN1.19
- net at CN1.2: now also C31.1
- net TP2: now reaches CN1.20
- net TP3: now reaches CN1.21
- net TP4: now reaches CN1.22
- net TP5: now reaches CN1.23
- net TP6: now reaches CN1.24
- net at CN1.3: now also C32.2
- net at CN1.4: now also C32.1
- net at CN1.9: now also R19.2
- net Button: no longer names the net of U1.18 (PB0)
- net EN1: no longer names the net of U1.10 (PA0)
- net ERROR: no longer names the net of U1.22 (PB11)
- net PWMA: no longer names the net of U1.29 (PA8)
- net SPI2_CS: no longer names the net of U1.25 (PB12)
- net SPI2_MISO renamed CFG2
- net CFG2: now also U7.2 (CFG2)
- net SPI2_MOSI renamed CFG3
- net CFG3: now also U7.3 (CFG3)
- net SPI2_SCK renamed CFG1
- net CFG1: now also U7.9 (CFG1)
- net USART2_RX: no longer names the net of U1.13 (PA3)
- net USART2_TX: no longer names the net of U1.12 (PA2)
- new net: C33.1, R21.1
- new net: R20.2, R22.1, R24.1
- new net: R16.1, U7.8 (VBUS)
- new net: C18.1, R14.2, R15.1
- new net: C17.1, R13.2, U7.1 (VDD)
- new net: Q2.1 (B), R14.1
- new net: C16.1, Q2.3 (C), R12.2
- new net: C9.1, R4.1, R6.1, U3.1
- new net: C9.2, R4.2, R5.1, U3.4 (-)
- new net: C15.1, R10.1, R9.2
- new net: C12.1, R5.2
- new net: R8.1, U3.3 (+)
- new net B: U3.2 (V-)
- new net Board_Temp: R7.2
- new net Tip_Control: C18.2
- new net Tip_Temp: R6.2
- no-connect marks 15 -> 19
Other:
- moved on the sheet: C10, C11, CN1, J1, Q1, U2, U4, U5, U6

Commit message: update
Parts:
- added R26, R27: 10K/1%, Resistor_SMD:R_0402_1005Metric, symbol Device:R_Small
- added SW1, SW2: SW_Push, Button_Switch_SMD:SW_SPST_PTS810, symbol Switch:SW_Push
- J2: value Conn_01x04 -> Negative
- J3: value Conn_01x04 -> Positive
- J7: value Conn_01x04 -> Com
Connections:
- net A: now also J3.1 (Pin_1), J3.2 (Pin_2), J3.3 (Pin_3), J3.4 (Pin_4), J6.1 (Pin_1), J6.2 (Pin_2), J6.3 (Pin_3), J6.4 (Pin_4)
- net B: now also J2.1 (Pin_1), J2.2 (Pin_2), J2.3 (Pin_3), J2.4 (Pin_4), J5.1 (Pin_1), J5.2 (Pin_2), J5.3 (Pin_3), J5.4 (Pin_4)
- net Board_Temp: now also U1.12 (PA2)
- net GND: now also CN1.25, CN1.26, CN1.27, CN1.28, J4.1 (Pin_1), J4.2 (Pin_2), J4.3 (Pin_3), J4.4 (Pin_4), J7.1 (Pin_1), J7.2 (Pin_2), J7.3 (Pin_3), J7.4 (Pin_4), SW1.2, SW2.2
- net Tip_Control: now also U1.13 (PA3)
- net Tip_Temp: now also U1.11 (PA1)
- net INT2: now reaches U2.11 (INT2)
- net INT2: now also U1.33 (PA12)
- net INT1: now reaches U2.12 (INT1)
- net INT1: now also U1.32 (PA11)
- net Vin_Sense: now reaches C15.1, R10.1, R9.2
- net Vin_Sense: now also U1.10 (PA0)
- net Button1: now reaches U1.22 (PB11)
- net Button1: now also R26.1
- net Button2: now reaches U1.25 (PB12)
- net Button2: now also R27.1
- new net: R26.2, SW1.1
- new net: R27.2, SW2.1
Other:
- note added: "Cold junction compensation"
- note added: "Interface"
- note added: "Power"
- note added: "Tip_Control"
- note added: "USART"
- moved on the sheet: C10, C11, C12, C13, C14, C15, C16, C17, C18, C19, C20, C21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

Commit message: update
Parts:
- removed C1, C4: 30PF, Capacitor_SMD:C_0402_1005Metric, symbol Device:C_Small
Changed lines of the file:
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@@
   (junction (at 180.34 62.23) (diameter 0) (color 0 0 0 0)
   )
-  (junction (at 43.942 125.476) (diameter 0) (color 0 0 0 0)
-  )
   (junction (at 44.45 204.47) (diameter 0) (color 0 0 0 0)
   )
@@
   (junction (at 259.08 248.92) (diameter 0) (color 0 0 0 0)
   )
-  (junction (at 33.528 125.476) (diameter 0) (color 0 0 0 0)
-  )
   (junction (at 109.22 267.97) (diameter 0) (color 0 0 0 0)
   )
@@
   (junction (at 78.74 260.35) (diameter 0) (color 0 0 0 0)
   )
-  (junction (at 33.528 136.271) (diameter 0) (color 0 0 0 0)
-  )
   (junction (at 33.782 86.36) (diameter 0) (color 0 0 0 0)
   )
@@
     (stroke (width 0) (type default) (color 0 0 0 0))
   )
-  (wire (pts (xy 38.608 136.271) (xy 33.528 136.271))
-    (stroke (width 0) (type default) (color 0 0 0 0))
-  )
   (wire (pts (xy 101.6 142.24) (xy 104.648 142.24))
     (stroke (width 0) (type default) (color 0 0 0 0))
@@
     (stroke (width 0) (type default) (color 0 0 0 0))
   )
-  (wire (pts (xy 33.528 136.906) (xy 33.528 136.271))
-    (stroke (width 0) (type default) (color 0 0 0 0))
-  )
   (wire (pts (xy 360.68 228.6) (xy 358.14 228.6))
     (stroke (width 0) (type default) (color 0 0 0 0))
@@
     (stroke (width 0) (type default) (color 0 0 0 0))
   )
-  (wire (pts (xy 43.942 136.906) (xy 43.942 134.366))
-    (stroke (width 0) (type default) (color 0 0 0 0))
-  )
   (wire (pts (xy 161.29 113.03) (xy 161.29 119.38))
     (stroke (width 0) (type default) (color 0 0 0 0))
@@
     (stroke (width 0) (type default) (color 0 0 0 0))
   )
-  (wire (pts (xy 38.608 128.016) (xy 38.608 136.271))
-    (stroke (width 0) (type default) (color 0 0 0 0))
-  )
   (wire (pts (xy 175.26 123.19) (xy 167.64 123.19))
     (stroke (width 0) (type default) (color 0 0 0 0))
@@
     (stroke (width 0) (type default) (color 0 0 0 0))
   )
-  (wire (pts (xy 33.528 125.476) (xy 33.528 129.286))
-    (stroke (width 0) (type default) (color 0 0 0 0))
-  )
   (wire (pts (xy 360.68 220.98) (xy 328.93 220.98))
     (stroke (width 0) (type default) (color 0 0 0 0))
@@
     (stroke (width 0) (type default) (color 0 0 0 0))
   )
-  (wire (pts (xy 43.942 125.476) (xy 43.942 129.286))
-    (stroke (width 0) (type default) (color 0 0 0 0))
-  )
-  (wire (pts (xy 33.528 136.271) (xy 33.528 134.366))
-    (stroke (width 0) (type default) (color 0 0 0 0))
-  )
   (wire (pts (xy 214.63 243.84) (xy 214.63 246.38))
     (stroke (width 0) (type default) (color 0 0 0 0))
@@
     (stroke (width 0) (type default) (color 0 0 0 0))
   )
+  (wire (pts (xy 38.608 128.016) (xy 38.608 129.794))
+    (stroke (width 0) (type default) (color 0 0 0 0))
+  )
   (wire (pts (xy 83.82 153.416) (xy 86.36 153.416))
     (stroke (width 0) (type default) (color 0 0 0 0))
@@
     (pin "2")
   )
-  (symbol (lib_id "Device:C_Small") (at 43.942 131.826 0) (unit 1)
-    (in_bom yes) (on_board yes)
-    (property "Reference" "C4" (id 0) (at 46.2788 130.6576 0)
-      (effects (font (size 1.27 1.27)) (justify left))
-    )
-    (property "Value" "30PF" (id 1) (at 46.2788 132.969 0)
-      (effects (font (size 1.27 1.27)) (justify left))
-    )
-    (property "Footprint" "Capacitor_SMD:C_0402_1005Metric" (id 2) (at 43.942 131.826 0)
-      (effects (font (size 1.27 1.27)) hide)
-    )
-    (property "Datasheet" "~" (id 3) (at 43.942 131.826 0)
-      (effects (font (size 1.27 1.27)) hide)
-    )
-    (pin "1")
-    (pin "2")
-  )
   (symbol (lib_id "Transistor_BJT:MMBT3904") (at 76.2 212.09 0) (mirror y) (unit 1)
     (in_bom yes) (on_board yes)
@@
     (pin "1")
   )
-  (symbol (lib_id "power:GND") (at 33.528 136.906 0) (unit 1)
+  (symbol (lib_id "power:GND") (at 38.608 129.794 0) (unit 1)
     (in_bom yes) (on_board yes)
-    (property "Reference" "#PWR0102" (id 0) (at 33.528 143.256 0)
+    (property "Reference" "#PWR0102" (id 0) (at 38.608 136.144 0)
       (effects (font (size 1.27 1.27)) hide)
     )
-    (property "Value" "GND" (id 1) (at 33.655 141.3002 0))
-    (property "Footprint" "" (id 2) (at 33.528 136.906 0)
+    (property "Value" "GND" (id 1) (at 38.735 134.1882 0))
+    (property "Footprint" "" (id 2) (at 38.608 129.794 0)
       (effects (font (size 1.27 1.27)) hide)
     )
-    (property "Datasheet" "" (id 3) (at 33.528 136.906 0)
+    (property "Datasheet" "" (id 3) (at 38.608 129.794 0)
       (effects (font (size 1.27 1.27)) hide)
     )
@@
     (pin "2")
   )
-  (symbol (lib_id "power:GND") (at 43.942 136.906 0) (unit 1)
-    (in_bom yes) (on_board yes)
-    (property "Reference" "#PWR0103" (id 0) (at 43.942 143.256 0)
-      (effects (font (size 1.27 1.27)) hide)
-    )
-    (property "Value" "GND" (id 1) (at 44.069 141.3002 0))
-    (property "Footprint" "" (id 2) (at 43.942 136.906 0)
-      (effects (font (size 1.27 1.27)) hide)
-    )
-    (property "Datasheet" "" (id 3) (at 43.942 136.906 0)
-      (effects (font (size 1.27 1.27)) hide)
-    )
-    (pin "1")
-  )
   (symbol (lib_id "Device:C_Small") (at 59.69 214.63 0) (unit 1)
     (in_bom yes) (on_board yes) (fields_autoplaced)
@@
     (pin "2")
   )
-  (symbol (lib_id "Device:C_Small") (at 33.528 131.826 0) (unit 1)
-    (in_bom yes) (on_board yes)
-    (property "Reference" "C1" (id 0) (at 35.8648 130.6576 0)
-      (effects (font (size 1.27 1.27)) (justify left))
-    )
-    (property "Value" "30PF" (id 1) (at 35.8648 132.969 0)
-      (effects (font (size 1.27 1.27)) (justify left))
-    )
-    (property "Footprint" "Capacitor_SMD:C_0402_1005Metric" (id 2) (at 33.528 131.826 0)
-      (effects (font (size 1.27 1.27)) hide)
-    )
-    (property "Datasheet" "~" (id 3) (at 33.528 131.826 0)
-      (effects (font (size 1.27 1.27)) hide)
-    )
-    (pin "1")
-    (pin "2")
-  )
   (symbol (lib_id "Device:R_Small") (at 158.75 121.92 90) (unit 1)
     (in_bom yes) (on_board yes)
@@
       (reference "#PWR0102") (unit 1) (value "GND") (footprint "")
     )
-    (path "/6c29f336-b70a-441f-abe5-9e2e6de721d4"
-      (reference "#PWR0103") (unit 1) (value "GND") (footprint "")
-    )
     (path "/c3599fdc-fa7a-4fa9-ae64-07850e64f222"
       (reference "#PWR0104") (unit 1) (value "GND") (footprint "")
@@
       (reference "#PWR0146") (unit 1) (value "GND") (footprint "")
     )
-    (path "/d53051b6-ebe9-4558-9887-00e35561baeb"
-      (reference "C1") (unit 1) (value "30PF") (footprint "Capacitor_SMD:C_0402_1005Metric")
-    )
     (path "/16204e20-03a6-43f4-b0bd-9183ea06dcf0"
       (reference "C2") (unit 1) (value "4u7") (footprint "Capacitor_SMD:C_0402_1005Metric")
@@
       (reference "C3") (unit 1) (value "100nf") (footprint "Capacitor_SMD:C_0402_1005Metric")
     )
-    (path "/1e0c06d7-8030-431f-903f-0bb75e65aa9c"
-      (reference "C4") (unit 1) (value "30PF") (footprint "Capacitor_SMD:C_0402_1005Metric")
-    )
     (path "/78282128-dde4-4902-bb1a-f3490742fc95"

Commit message: PCB layout update
Parts:
- added C1: 1uF, Capacitor_SMD:C_0402_1005Metric, symbol Device:C_Small
- added J8: Conn_01x04, Connector_JST:JST_SH_BM04B-SRSS-TB_1x04-1MP_P1.00mm_Vertical, symbol Connector_Generic:Conn_01x04
- added R28: 50K, Resistor_SMD:R_0402_1005Metric, symbol Device:R_Small
- added R29: 9K, Resistor_SMD:R_0402_1005Metric, symbol Device:R_Small
Connections:
- net MISO is gone; now on net RESET: U1.16 (PA6)
- net MOSI is gone; now on net SDA: U1.17 (PA7)
- net +1V8: now also C1.2
- net +3V3: now also J8.1 (Pin_1)
- net Button1: now also U1.43 (PB7); no longer U1.22 (PB11)
- net Button2: now also U1.45 (PB8); no longer U1.25 (PB12)
- net CFG1: now also U1.46 (PB9); no longer U1.26 (PB13)
- net CFG2: now also U1.21 (PB10); no longer U1.27 (PB14)
- net CFG3: now also U1.22 (PB11); no longer U1.28 (PB15)
- net DCX: now also U1.29 (PA8)
- net GND: now also C1.1, J8.4 (Pin_4), R29.1
- net INT1: now also U1.42 (PB6); no longer U1.32 (PA11)
- net INT2: now also U1.41 (PB5); no longer U1.33 (PA12)
- net SCL: now also U1.15 (PA5); no longer U1.42 (PB6)
- net SDA: no longer U1.43 (PB7), U2.4 (SDA/SDI)
- net SWCLK: now also J8.2 (Pin_2)
- net SWDIO: now also J8.3 (Pin_3)
- net VBUS: now also R28.2
- net Voltage: now reaches U1.18 (PB0)
- net Voltage: now also R28.1, R29.2
- net CS renamed DISPLAY_CS
- net DISPLAY_CS: no longer U2.2 (~{CS})
- net SCK renamed IMU_SCK
- net IMU_SCK: now also U1.26 (PB13); no longer U1.15 (PA5)
- net SD0 renamed IMU_SD0
- net IMU_SD0: now also U1.27 (PB14)
- new net IMU_CS: U1.25 (PB12), U2.2 (~{CS})
- new net IMU_SDA: U1.28 (PB15), U2.4 (SDA/SDI)
- no-connect marks 19 -> 17
Other:
- moved on the sheet: C22

Commit message: PCB layout update
Parts:
- added C36, C37: 100nF, Capacitor_SMD:C_0402_1005Metric, symbol Device:C_Small
- added C4: 1uf, Capacitor_SMD:C_0402_1005Metric, symbol Device:C_Small
- added R30, R31, R32, R33, R34, R35, R36: 10K/1%, Resistor_SMD:R_0402_1005Metric, symbol Device:R_Small
- added U10: TXS0102DCU, Package_SO:VSSOP-8_2.3x2mm_P0.5mm, symbol Logic_LevelTranslator:TXS0102DCU
Connections:
- net +1V8: now also C36.2, C4.2, R30.1, R31.1, R32.2, R33.2, R34.2, U10.3 (VCCA), U10.6 (OE)
- net +3V3: now also C37.2, R35.1, R36.1, U10.7 (VCCB)
- net Button1: now also U1.4 (PC15); no longer U1.43 (PB7)
- net Button2: now also U1.3 (PC14); no longer U1.45 (PB8)
- net CFG1: now also U1.41 (PB5); no longer U1.46 (PB9)
- net CFG2: now also U1.42 (PB6); no longer U1.21 (PB10)
- net CFG3: now also U1.43 (PB7); no longer U1.22 (PB11)
- net GND: now also C36.1, C37.1, C4.1, U10.2 (GND)
- net IMU_CS: now also R34.1; no longer U1.25 (PB12)
- net INT1: now also U1.45 (PB8), R33.1; no longer U1.42 (PB6)
- net INT2: now also U1.46 (PB9), R32.1; no longer U1.41 (PB5)
- net Voltage: no longer U1.18 (PB0)
- net IMU_SCK: no longer names the net of U1.26 (PB13)
- net IMU_SCK: no longer U2.1 (SCL/SPC)
- net IMU_SD0: no longer names the net of U1.27 (PB14)
- net IMU_SD0: no longer U2.3 (SA0/SDO)
- net IMU_SDA: no longer names the net of U1.28 (PB15)
- net IMU_SDA: no longer U2.4 (SDA/SDI)
- new net IMU_SCL_1.8V: R31.2, U10.5 (A1), U2.1 (SCL/SPC)
- new net IMU_SCL_3.3V: R36.2, U1.21 (PB10), U10.8 (B1)
- new net IMU_SD0_1.8V: U2.3 (SA0/SDO)
- new net IMU_SDA_1.8V: R30.2, U10.4 (A2), U2.4 (SDA/SDI)
- new net IMU_SDA_3.3V: R35.2, U1.22 (PB11), U10.1 (B2)
- no-connect marks 17 -> 20
Other:
- moved on the sheet: C22, C26, C29, C30, C31, C32, CN1, R19, R23, R25, R26, R27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

Commit message: PCB layout update
Parts:
- removed C10, C11: 100nf, Capacitor_SMD:C_0402_1005Metric_Pad0.74x0.62mm_HandSolder, symbol Device:C_Small
- removed J8: Conn_01x04, Connector_JST:JST_SH_BM04B-SRSS-TB_1x04-1MP_P1.00mm_Vertical, symbol Connector_Generic:Conn_01x04
- removed R28: 50K, Resistor_SMD:R_0402_1005Metric, symbol Device:R_Small
- removed R29: 9K, Resistor_SMD:R_0402_1005Metric, symbol Device:R_Small
- removed U5: CH340E, Package_SO:MSOP-10_3x3mm_P0.5mm, symbol Interface_USB:CH340E
- added J8: Conn_01x06, Connector_JST:JST_SH_BM06B-SRSS-TB_1x06-1MP_P1.00mm_Vertical, symbol Connector_Generic:Conn_01x06
Connections:
- net +3V3: now also J8.1 (Pin_1)
- net GND: now also J8.6 (Pin_6)
- net SWCLK: now also J8.2 (Pin_2)
- net SWDIO: now also J8.3 (Pin_3)
- net USART_RX: now also J8.5 (Pin_5)
- net USART_TX: now also J8.4 (Pin_4)
- no-connect marks 20 -> 17
Other:
- note removed: "USART"
